File: fruity60/fruity60.sch (KiCad schematic (older format))
At the start: 126 parts

Commit message: Update schematic and silkscreen
Parts:
- MX0: value MX-NoLED -> K00
- MX0A1: value MX-NoLED -> K0A
- MX1: value MX-NoLED -> K01
- MX10: value MX-NoLED -> K10
- MX11: value MX-NoLED -> K11
- MX12: value MX-NoLED -> K12
- MX13: value MX-NoLED -> K13
- MX14: value MX-NoLED -> K14
- MX15: value MX-NoLED -> K15
- MX16: value MX-NoLED -> K16
- MX17: value MX-NoLED -> K17
- MX18: value MX-NoLED -> K18
- MX19: value MX-NoLED -> K19
- MX1A1: value MX-NoLED -> K1A
- MX2: value MX-NoLED -> K02
- MX20: value MX-NoLED -> K20
- MX21: value MX-NoLED -> K21
- MX22: value MX-NoLED -> K22
- MX23: value MX-NoLED -> K23
- MX24: value MX-NoLED -> K24
- MX25: value MX-NoLED -> K25
- MX26: value MX-NoLED -> K26
- MX27: value MX-NoLED -> K27
- MX28: value MX-NoLED -> K28
- MX29: value MX-NoLED -> K29
- MX2A1: value MX-NoLED -> K2A
- MX3: value MX-NoLED -> K03
- MX30: value MX-NoLED -> K30
- MX31: value MX-NoLED -> K31
- MX32: value MX-NoLED -> K32
- MX33: value MX-NoLED -> K33
- MX34: value MX-NoLED -> K34
- MX35: value MX-NoLED -> K35
- MX36: value MX-NoLED -> K36
- MX37: value MX-NoLED -> K37
- MX38: value MX-NoLED -> K38
- MX39: value MX-NoLED -> K39
- MX3A1: value MX-NoLED -> K3A
- MX4: value MX-NoLED -> K04
- MX40: value MX-NoLED -> K40
- MX41: value MX-NoLED -> K41
- MX42: value MX-NoLED -> K42
- MX45: value MX-NoLED -> K45
- MX48: value MX-NoLED -> K48
- MX49: value MX-NoLED -> K49
- MX4A1: value MX-NoLED -> K4A
- MX5: value MX-NoLED -> K05
- MX50: value MX-NoLED -> K50
- MX51: value MX-NoLED -> K51
- MX52: value MX-NoLED -> K52
- MX53: value MX-NoLED -> K53
- MX54: value MX-NoLED -> K54
- MX55: value MX-NoLED -> K55
- MX56: value MX-NoLED -> K56
- MX57: value MX-NoLED -> K57
- MX58: value MX-NoLED -> K58
- MX59: value MX-NoLED -> K59
- MX5A1: value MX-NoLED -> K5A
- MX6: value MX-NoLED -> K06
- MX7: value MX-NoLED -> K07
- MX8: value MX-NoLED -> K08
- MX9: value MX-NoLED -> K09
